Commit message: ROS interface and simulation

File: workspace/limo_simulation/urdf/limo_ackerman.xacro (robot description, xacro)
@@ -28,5 +28,5 @@
             <origin xyz="0 0 -0.15" rpy="0 0 1.57" />
             <geometry>
-                <mesh filename="file://$(find limo_simulation)/meshes/limo_base.dae" scale="1 1 1"/>
+                <mesh filename="file://$(find limo_simulation)/meshes/limo_base.stl" scale="0.001 0.001 0.001"/>
             </geometry>
         </visual>
@@ -76,5 +76,5 @@
             <origin xyz="0 0 0" rpy="0 0 0" />
             <geometry>
-                <mesh filename="file://$(find limo_simulation)/meshes/limo_wheel.dae" />
+                <mesh filename="file://$(find limo_simulation)/meshes/limo_wheel.stl" scale="0.001 0.001 0.001"/>
             </geometry>
         </visual>
@@ -101,5 +101,5 @@
             <origin xyz="0 0 0" rpy="0 0 0" />
             <geometry>
-                <mesh filename="file://$(find limo_simulation)/meshes/limo_wheel.dae" />
+                <mesh filename="file://$(find limo_simulation)/meshes/limo_wheel.stl" scale="0.001 0.001 0.001"/>
             </geometry>
         </visual>

File: workspace/limo_simulation/urdf/limo_xacro.xacro (robot description, xacro)
@@ -11,5 +11,5 @@
                 <origin xyz="0 0 0" rpy="0 0 0" />
                 <geometry>
-                    <mesh filename="file://$(find limo_simulation)/meshes/limo_wheel.dae" />
+                    <mesh filename="file://$(find limo_simulation)/meshes/limo_wheel.stl" scale="0.001 0.001 0.001"/>
                 </geometry>
             </visual>
